File: pcb/BinaryClock.sch (KiCad schematic (older format))
At the start: 20 parts

Commit message: pcb layout begun
Parts:
- removed BT?: Battery_Cell, symbol Battery_Cell
- removed IC?: ATMEGA328-AU, TQFP32, symbol ATMEGA328-AU
- removed R? (x5): R_Small, symbol R_Small
- removed U?: ATmega32U4, symbol ATmega32U4
- removed U?: DS3231, Housings_SOIC:SOIC-16_7.5x10.3mm_Pitch1.27mm, symbol DS3231
- added CON1: AVR-ISP-6, Pin_Headers:Pin_Header_Straight_2x03_Pitch2.54mm, symbol AVR-ISP-6
- added IC1: ATMEGA328P-A, Housings_QFP:TQFP-44_10x10mm_Pitch0.8mm, symbol ATMEGA328P-A
- added U1: LM78M05CT, Power_Integrations:TO-220, symbol LM78M05CT
- added U3, U4, U5: clock_header, Pin_Headers:Pin_Header_Straight_1x03_Pitch2.54mm, symbol clock_header
- C1, C2, C3: renamed from C?; footprint (none) -> Capacitors_SMD:C_0805
- R1, R2, R3, R4, R5: renamed from R?; footprint (none) -> Resistors_SMD:R_0805
- Y1: renamed from Y?; footprint (none) -> Crystals:Crystal_HC18-U_Horizontal
- gave numbers to parts that had none: 2
Connections:
- net labels added: MISO, MOSI, RESET, SCK, VIN
- net labels removed: +5V
- wire segments 53 -> 76
Other:
- moved on the sheet: BT1, R4, R5, U2

Commit message: Progress toward high level board layout. Board is still missing a voltage reulator
Parts:
- removed U1: LM78M05CT, Power_Integrations:TO-220, symbol LM78M05CT
- added U1: TPS7150QD, SO-8, symbol TPS7150QD
Changed lines of the file:
@@
 LIBS:maxim
 LIBS:binaryclock
+LIBS:BinaryClock-cache
 EELAYER 25 0
 EELAYER END
@@
 	2750 3350 2400 3350
 $Comp
-L LM78M05CT U1
-U 1 1 589165BE
-P 2300 1450
-F 0 "U1" H 2100 1650 50  0000 C CNN
-F 1 "LM78M05CT" H 2300 1650 50  0000 L CNN
-F 2 "Power_Integrations:TO-220" H 2300 1550 50  0000 C CIN
-F 3 "" H 2300 1450 50  0000 C CNN
-	1    2300 1450
-	1    0    0    -1
-$EndComp
-Text Label 1700 1400 2    60   ~ 0
-VIN
-Wire Wire Line
-	1700 1400 1900 1400
-$Comp
-L VCC #PWR011
-U 1 1 58916735
-P 2900 1300
-F 0 "#PWR011" H 2900 1150 50  0001 C CNN
-F 1 "VCC" H 2900 1450 50  0000 C CNN
-F 2 "" H 2900 1300 50  0000 C CNN
-F 3 "" H 2900 1300 50  0000 C CNN
-	1    2900 1300
-	1    0    0    -1
-$EndComp
-Wire Wire Line
-	2900 1300 2900 1400
-Wire Wire Line
-	2900 1400 2700 1400
-$Comp
-L GND #PWR012
-U 1 1 589167B9
-P 2300 1850
-F 0 "#PWR012" H 2300 1600 50  0001 C CNN
-F 1 "GND" H 2300 1700 50  0000 C CNN
-F 2 "" H 2300 1850 50  0000 C CNN
-F 3 "" H 2300 1850 50  0000 C CNN
-	1    2300 1850
-	1    0    0    -1
-$EndComp
-Wire Wire Line
-	2300 1850 2300 1700
-$Comp
 L clock_header U3
 U 1 1 58ACEEBD
@@
 	10000 2750 9800 2750
 $Comp
-L VCC #PWR013
+L VCC #PWR011
 U 1 1 58ACF519
 P 9250 1250
-F 0 "#PWR013" H 9250 1100 50  0001 C CNN
+F 0 "#PWR011" H 9250 1100 50  0001 C CNN
 F 1 "VCC" H 9250 1400 50  0000 C CNN
 F 2 "" H 9250 1250 50  0000 C CNN
@@
 $EndComp
 $Comp
-L GND #PWR014
+L GND #PWR012
 U 1 1 58ACF56C
 P 9400 3100
-F 0 "#PWR014" H 9400 2850 50  0001 C CNN
+F 0 "#PWR012" H 9400 2850 50  0001 C CNN
 F 1 "GND" H 9400 2950 50  0000 C CNN
 F 2 "" H 9400 3100 50  0000 C CNN
@@
 Connection ~ 9250 1550
 Wire Wire Line
-	9400 3100 9400 1650
+	9400 1650 9400 3100
 Wire Wire Line
 	9400 1650 9950 1650
@@
 	8250 5100 8950 5100
 Connection ~ 8550 4050
+$Comp
+L TPS7150QD U1
+U 1 1 58AE7B9A
+P 2250 1650
+F 0 "U1" H 1950 2000 50  0000 C CNN
+F 1 "TPS7150QD" H 2450 2000 50  0000 C CNN
+F 2 "SO-8" H 2250 1650 50  0000 C CIN
+F 3 "" H 2250 1650 50  0000 C CNN
+	1    2250 1650
+	1    0    0    -1
+$EndComp
+$Comp
+L GND #PWR013
+U 1 1 58AEEE1E
+P 2250 2350
+F 0 "#PWR013" H 2250 2100 50  0001 C CNN
+F 1 "GND" H 2250 2200 50  0000 C CNN
+F 2 "" H 2250 2350 50  0000 C CNN
+F 3 "" H 2250 2350 50  0000 C CNN
+	1    2250 2350
+	1    0    0    -1
+$EndComp
+Wire Wire Line
+	2250 2100 2250 2350
+$Comp
+L VCC #PWR014
+U 1 1 58AEEFF6
+P 3000 1100
+F 0 "#PWR014" H 3000 950 50  0001 C CNN
+F 1 "VCC" H 3000 1250 50  0000 C CNN
+F 2 "" H 3000 1100 50  0000 C CNN
+F 3 "" H 3000 1100 50  0000 C CNN
+	1    3000 1100
+	1    0    0    -1
+$EndComp
+Text Label 1350 1450 2    60   ~ 0
+VIN
+Wire Wire Line
+	1350 1450 1750 1450
+Wire Wire Line
+	2750 1450 3000 1450
+Wire Wire Line
+	3000 1450 3000 1100
 $EndSCHEMATC

Commit message: Added voltage regulator to pcb schematic and layout. Started routing on the board layout
Parts:
- removed C1: C, Capacitors_SMD:C_0805, symbol C
- removed U1: TPS7150QD, SO-8, symbol TPS7150QD
- added R6: 10K, symbol R
- added U1: MC33269, tapMatrix_Shield:SOT223_318H, symbol MC33269
Connections:
- wire segments 76 -> 77
Changed lines of the file:
@@
 $EndComp
 $Comp
-L GND #PWR01
+L GND #PWR7
 U 1 1 5887FC8B
 P 7900 3550
-F 0 "#PWR01" H 7900 3300 50  0001 C CNN
+F 0 "#PWR7" H 7900 3300 50  0001 C CNN
 F 1 "GND" H 7900 3400 50  0000 C CNN
 F 2 "" H 7900 3550 50  0000 C CNN
@@
 $EndComp
 $Comp
-L VCC #PWR02
+L VCC #PWR5
 U 1 1 5888112B
 P 4050 1900
-F 0 "#PWR02" H 4050 1750 50  0001 C CNN
+F 0 "#PWR5" H 4050 1750 50  0001 C CNN
 F 1 "VCC" H 4050 2050 50  0000 C CNN
 F 2 "" H 4050 1900 50  0000 C CNN
@@
 $EndComp
 $Comp
-L GND #PWR03
+L GND #PWR13
 U 1 1 588813DC
 P 9450 5550
-F 0 "#PWR03" H 9450 5300 50  0001 C CNN
+F 0 "#PWR13" H 9450 5300 50  0001 C CNN
 F 1 "GND" H 9450 5400 50  0000 C CNN
 F 2 "" H 9450 5550 50  0000 C CNN
@@
 $EndComp
 $Comp
-L GND #PWR04
+L GND #PWR14
 U 1 1 5888182A
 P 10250 5550
-F 0 "#PWR04" H 10250 5300 50  0001 C CNN
+F 0 "#PWR14" H 10250 5300 50  0001 C CNN
 F 1 "GND" H 10250 5400 50  0000 C CNN
 F 2 "" H 10250 5550 50  0000 C CNN
@@
 $EndComp
 $Comp
-L VCC #PWR05
+L VCC #PWR12
 U 1 1 588818D8
 P 9450 4400
-F 0 "#PWR05" H 9450 4250 50  0001 C CNN
+F 0 "#PWR12" H 9450 4250 50  0001 C CNN
 F 1 "VCC" H 9450 4550 50  0000 C CNN
 F 2 "" H 9450 4400 50  0000 C CNN
@@
 SDA
 $Comp
-L VCC #PWR06
+L VCC #PWR8
 U 1 1 5888547F
 P 8550 3950
-F 0 "#PWR06" H 8550 3800 50  0001 C CNN
+F 0 "#PWR8" H 8550 3800 50  0001 C CNN
 F 1 "VCC" H 8550 4100 50  0000 C CNN
 F 2 "" H 8550 3950 50  0000 C CNN
@@
 $EndComp
 $Comp
-L VCC #PWR07
+L VCC #PWR9
 U 1 1 588854C3
 P 8850 3950
-F 0 "#PWR07" H 8850 3800 50  0001 C CNN
+F 0 "#PWR9" H 8850 3800 50  0001 C CNN
 F 1 "VCC" H 8850 4100 50  0000 C CNN
 F 2 "" H 8850 3950 50  0000 C CNN
@@
 $EndComp
 $Comp
-L GND #PWR08
+L GND #PWR6
 U 1 1 58885855
 P 4100 4800
-F 0 "#PWR08" H 4100 4550 50  0001 C CNN
+F 0 "#PWR6" H 4100 4550 50  0001 C CNN
 F 1 "GND" H 4100 4650 50  0000 C CNN
 F 2 "" H 4100 4800 50  0000 C CNN
@@
 	1    0    0    -1
 $EndComp
-$Comp
-L C C1
-U 1 1 58885A9D
-P 4100 3200
-F 0 "C1" H 4125 3300 50  0000 L CNN
-F 1 "C" H 4125 3100 50  0000 L CNN
-F 2 "Capacitors_SMD:C_0805" H 4138 3050 50  0001 C CNN
-F 3 "" H 4100 3200 50  0000 C CNN
-	1    4100 3200
-	1    0    0    -1
-$EndComp
 Wire Wire Line
 	7950 4800 8950 4800
@@
 	4400 4350 4100 4350
 Wire Wire Line
-	4100 3350 4100 4800
-Wire Wire Line
 	4400 4450 4100 4450
 Connection ~ 4100 4450
 Wire Wire Line
-	4400 4550 4100 4550
+	4100 4550 4400 4550
 Connection ~ 4100 4550
-Wire Wire Line
-	4400 2850 4100 2850
-Wire Wire Line
-	4100 2850 4100 3050
 Connection ~ 4100 4350
 Wire Wire Line
@@
 Text Label 1750 3150 2    60   ~ 0
 MISO
-Text Label 6400 3750 0    60   ~ 0
+Text Label 6550 3700 0    60   ~ 0
 RESET
-Wire Wire Line
-	6300 3700 6350 3700
-Wire Wire Line
-	6350 3700 6350 3750
-Wire Wire Line
-	6350 3750 6400 3750
 Wire Wire Line
 	6300 2750 6350 2750
@@
 Text Label 2800 3250 0    60   ~ 0
 MOSI
-Text Label 1750 3350 2    60   ~ 0
+Text Label 1000 3350 2    60   ~ 0
 RESET
 Wire Wire Line
@@
 	2150 3250 1750 3250
 Wire Wire Line
-	1750 3350 2150 3350
+	1000 3350 2150 3350
 Wire Wire Line
 	2400 3250 2800 3250
 $Comp
-L VCC #PWR09
+L VCC #PWR2
 U 1 1 5891639F
-P 2750 2900
-F 0 "#PWR09" H 2750 2750 50  0001 C CNN
-F 1 "VCC" H 2750 3050 50  0000 C CNN
-F 2 "" H 2750 2900 50  0000 C CNN
-F 3 "" H 2750 2900 50  0000 C CNN
-	1    2750 2900
-	1    0    0    -1
-$EndComp
-Wire Wire Line
-	2750 2900 2750 3150
+P 2750 2650
+F 0 "#PWR2" H 2750 2500 50  0001 C CNN
+F 1 "VCC" H 2750 2800 50  0000 C CNN
+F 2 "" H 2750 2650 50  0000 C CNN
+F 3 "" H 2750 2650 50  0000 C CNN
+	1    2750 2650
+	1    0    0    -1
+$EndComp
+Wire Wire Line
+	2750 2650 2750 3150
 Wire Wire Line
 	2750 3150 2400 3150
 $Comp
-L GND #PWR010
+L GND #PWR3
 U 1 1 5891641C
 P 2750 3600
-F 0 "#PWR010" H 2750 3350 50  0001 C CNN
+F 0 "#PWR3" H 2750 3350 50  0001 C CNN
 F 1 "GND" H 2750 3450 50  0000 C CNN
 F 2 "" H 2750 3600 50  0000 C CNN
@@
 	10000 2750 9800 2750
 $Comp
-L VCC #PWR011
+L VCC #PWR10
 U 1 1 58ACF519
 P 9250 1250
-F 0 "#PWR011" H 9250 1100 50  0001 C CNN
+F 0 "#PWR10" H 9250 1100 50  0001 C CNN
 F 1 "VCC" H 9250 1400 50  0000 C CNN
 F 2 "" H 9250 1250 50  0000 C CNN
@@
 $EndComp
 $Comp
-L GND #PWR012
+L GND #PWR11
 U 1 1 58ACF56C
 P 9400 3100
-F 0 "#PWR012" H 9400 2850 50  0001 C CNN
+F 0 "#PWR11" H 9400 2850 50  0001 C CNN
 F 1 "GND" H 9400 2950 50  0000 C CNN
 F 2 "" H 9400 3100 50  0000 C CNN
@@
 Connection ~ 8550 4050
 $Comp
-L TPS7150QD U1
-U 1 1 58AE7B9A
-P 2250 1650
-F 0 "U1" H 1950 2000 50  0000 C CNN
-F 1 "TPS7150QD" H 2450 2000 50  0000 C CNN
-F 2 "SO-8" H 2250 1650 50  0000 C CIN
-F 3 "" H 2250 1650 50  0000 C CNN
-	1    2250 1650
-	1    0    0    -1
-$EndComp
-$Comp
-L GND #PWR013
+L GND #PWR4
 U 1 1 58AEEE1E
-P 2250 2350
-F 0 "#PWR013" H 2250 2100 50  0001 C CNN
-F 1 "GND" H 2250 2200 50  0000 C CNN
-F 2 "" H 2250 2350 50  0000 C CNN
-F 3 "" H 2250 2350 50  0000 C CNN
-	1    2250 2350
-	1    0    0    -1
-$EndComp
-Wire Wire Line
-	2250 2100 2250 2350
-$Comp
-L VCC #PWR014
+P 2800 1850
+F 0 "#PWR4" H 2800 1600 50  0001 C CNN
+F 1 "GND" H 2800 1700 50  0000 C CNN
+F 2 "" H 2800 1850 50  0000 C CNN
+F 3 "" H 2800 1850 50  0000 C CNN
+	1    2800 1850
+	1    0    0    -1
+$EndComp
+Wire Wire Line
+	2000 1750 2000 2100
+$Comp
+L VCC #PWR1
 U 1 1 58AEEFF6
-P 3000 1100
-F 0 "#PWR014" H 3000 950 50  0001 C CNN
-F 1 "VCC" H 3000 1250 50  0000 C CNN
-F 2 "" H 3000 1100 50  0000 C CNN
-F 3 "" H 3000 1100 50  0000 C CNN
-	1    3000 1100
-	1    0    0    -1
-$EndComp
-Text Label 1350 1450 2    60   ~ 0
+P 2400 2000
+F 0 "#PWR1" H 2400 1850 50  0001 C CNN
+F 1 "VCC" H 2400 2150 50  0000 C CNN
+F 2 "" H 2400 2000 50  0000 C CNN
+F 3 "" H 2400 2000 50  0000 C CNN
+	1    2400 2000
+	1    0    0    -1
+$EndComp
+Text Label 1200 1450 2    60   ~ 0
 VIN
 Wire Wire Line
-	1350 1450 1750 1450
-Wire Wire Line
-	2750 1450 3000 1450
-Wire Wire Line
-	3000 1450 3000 1100
+	1200 1450 1600 1450
+Wire Wire Line
+	2400 1450 2800 1450
+Wire Wire Line
+	4100 4350 4100 4800
+$Comp
+L MC33269 U1
+U 1 1 58B6409C
+P 2000 1500
+F 0 "U1" H 1800 1700 50  0000 C CNN
+F 1 "MC33269" H 2000 1700 50  0000 L CNN
+F 2 "tapMatrix_Shield:SOT223_318H" H 2000 1600 50  0000 C CIN
+F 3 "" H 2000 1500 50  0000 C CNN
+	1    2000 1500
+	1    0    0    -1
+$EndComp
+Wire Wire Line
+	2000 2100 2400 2100
+Wire Wire Line
+	2400 2100 2400 2000
+Wire Wire Line
+	2800 1450 2800 1850
+Connection ~ 2650 1450
+Wire Wire Line
+	6550 3700 6300 3700
+Wire Wire Line
+	2750 2750 1300 2750
+Wire Wire Line
+	1300 2750 1300 2800
+Connection ~ 2750 2750
+$Comp
+L R R6
+U 1 1 58B6502D
+P 1300 2950
+F 0 "R6" V 1380 2950 50  0000 C CNN
+F 1 "10K" V 1300 2950 50  0000 C CNN
+F 2 "" V 1230 2950 50  0000 C CNN
+F 3 "" H 1300 2950 50  0000 C CNN
+	1    1300 2950
+	1    0    0    -1
+$EndComp
+Wire Wire Line
+	1300 3100 1300 3350
+Connection ~ 1300 3350
 $EndSCHEMATC

Commit message: Finished initial attempt at routing
Parts:
- added CON2: BARREL_JACK, Connectors:BARREL_JACK, symbol BARREL_JACK
- BT1: footprint (none) -> Battery_Holders:Keystone_3001_1x12mm-CoinCell
- U2: footprint Housings_SOIC:SOIC-16_7.5x10.3mm_Pitch1.27mm -> tapMatrix_Shield:DS3231
Connections:
- net GND: now also CON2.2
- net VCC: now also IC1.18 (AVCC); no longer U2.4 (~RST), U3.2 (power), U4.2 (power), U5.2 (power)
- net VIN: now also U3.2 (power), U4.2 (power), U5.2 (power), CON2.1
Other:
- moved on the sheet: U1
Changed lines of the file:
@@
 F 0 "U2" H 9350 5375 50  0000 R CNN
 F 1 "DS3231" H 9350 5300 50  0000 R CNN
-F 2 "Housings_SOIC:SOIC-16_7.5x10.3mm_Pitch1.27mm" H 9500 4500 50  0001 L CNN
+F 2 "tapMatrix_Shield:DS3231" H 9500 4500 50  0001 L CNN
 F 3 "" H 9720 5150 50  0001 C CNN
 	1    9450 4900
@@
 $EndComp
 $Comp
-L GND #PWR7
+L GND #PWR01
 U 1 1 5887FC8B
 P 7900 3550
-F 0 "#PWR7" H 7900 3300 50  0001 C CNN
+F 0 "#PWR01" H 7900 3300 50  0001 C CNN
 F 1 "GND" H 7900 3400 50  0000 C CNN
 F 2 "" H 7900 3550 50  0000 C CNN
@@
 $EndComp
 $Comp
-L VCC #PWR5
+L VCC #PWR02
 U 1 1 5888112B
 P 4050 1900
-F 0 "#PWR5" H 4050 1750 50  0001 C CNN
+F 0 "#PWR02" H 4050 1750 50  0001 C CNN
 F 1 "VCC" H 4050 2050 50  0000 C CNN
 F 2 "" H 4050 1900 50  0000 C CNN
@@
 $EndComp
 $Comp
-L GND #PWR13
+L GND #PWR03
 U 1 1 588813DC
 P 9450 5550
-F 0 "#PWR13" H 9450 5300 50  0001 C CNN
+F 0 "#PWR03" H 9450 5300 50  0001 C CNN
 F 1 "GND" H 9450 5400 50  0000 C CNN
 F 2 "" H 9450 5550 50  0000 C CNN
@@
 F 0 "BT1" H 10350 5400 50  0000 L CNN
 F 1 "Battery_Cell" H 10350 5300 50  0000 L CNN
-F 2 "" V 10250 5360 50  0001 C CNN
+F 2 "Battery_Holders:Keystone_3001_1x12mm-CoinCell" V 10250 5360 50  0001 C CNN
 F 3 "" V 10250 5360 50  0000 C CNN
 	1    10250 5300
@@
 $EndComp
 $Comp
-L GND #PWR14
+L GND #PWR04
 U 1 1 5888182A
 P 10250 5550
-F 0 "#PWR14" H 10250 5300 50  0001 C CNN
+F 0 "#PWR04" H 10250 5300 50  0001 C CNN
 F 1 "GND" H 10250 5400 50  0000 C CNN
 F 2 "" H 10250 5550 50  0000 C CNN
@@
 $EndComp
 $Comp
-L VCC #PWR12
+L VCC #PWR05
 U 1 1 588818D8
 P 9450 4400
-F 0 "#PWR12" H 9450 4250 50  0001 C CNN
+F 0 "#PWR05" H 9450 4250 50  0001 C CNN
 F 1 "VCC" H 9450 4550 50  0000 C CNN
 F 2 "" H 9450 4400 50  0000 C CNN
@@
 SDA
 $Comp
-L VCC #PWR8
+L VCC #PWR06
 U 1 1 5888547F
 P 8550 3950
-F 0 "#PWR8" H 8550 3800 50  0001 C CNN
+F 0 "#PWR06" H 8550 3800 50  0001 C CNN
 F 1 "VCC" H 8550 4100 50  0000 C CNN
 F 2 "" H 8550 3950 50  0000 C CNN
@@
 $EndComp
 $Comp
-L VCC #PWR9
+L VCC #PWR07
 U 1 1 588854C3
 P 8850 3950
-F 0 "#PWR9" H 8850 3800 50  0001 C CNN
+F 0 "#PWR07" H 8850 3800 50  0001 C CNN
 F 1 "VCC" H 8850 4100 50  0000 C CNN
 F 2 "" H 8850 3950 50  0000 C CNN
@@
 $EndComp
 $Comp
-L GND #PWR6
+L GND #PWR08
 U 1 1 58885855
 P 4100 4800
-F 0 "#PWR6" H 4100 4550 50  0001 C CNN
+F 0 "#PWR08" H 4100 4550 50  0001 C CNN
 F 1 "GND" H 4100 4650 50  0000 C CNN
 F 2 "" H 4100 4800 50  0000 C CNN
@@
 	6600 2450 6300 2450
 Wire Wire Line
-	8550 3950 8550 4200
-Wire Wire Line
 	8550 4500 8550 4800
 Wire Wire Line
@@
 	8850 4500 8850 4900
 Wire Wire Line
-	4050 1900 4050 2350
+	4050 1900 4050 2550
 Wire Wire Line
 	4050 2350 4400 2350
@@
 	2400 3250 2800 3250
 $Comp
-L VCC #PWR2
+L VCC #PWR09
 U 1 1 5891639F
 P 2750 2650
-F 0 "#PWR2" H 2750 2500 50  0001 C CNN
+F 0 "#PWR09" H 2750 2500 50  0001 C CNN
 F 1 "VCC" H 2750 2800 50  0000 C CNN
 F 2 "" H 2750 2650 50  0000 C CNN
@@
 	2750 3150 2400 3150
 $Comp
-L GND #PWR3
+L GND #PWR010
 U 1 1 5891641C
 P 2750 3600
-F 0 "#PWR3" H 2750 3350 50  0001 C CNN
+F 0 "#PWR010" H 2750 3350 50  0001 C CNN
 F 1 "GND" H 2750 3450 50  0000 C CNN
 F 2 "" H 2750 3600 50  0000 C CNN
@@
 	10000 2750 9800 2750
 $Comp
-L VCC #PWR10
-U 1 1 58ACF519
-P 9250 1250
-F 0 "#PWR10" H 9250 1100 50  0001 C CNN
-F 1 "VCC" H 9250 1400 50  0000 C CNN
-F 2 "" H 9250 1250 50  0000 C CNN
-F 3 "" H 9250 1250 50  0000 C CNN
-	1    9250 1250
-	1    0    0    -1
-$EndComp
-$Comp
-L GND #PWR11
+L GND #PWR011
 U 1 1 58ACF56C
 P 9400 3100
-F 0 "#PWR11" H 9400 2850 50  0001 C CNN
+F 0 "#PWR011" H 9400 2850 50  0001 C CNN
 F 1 "GND" H 9400 2950 50  0000 C CNN
 F 2 "" H 9400 3100 50  0000 C CNN
@@
 Text GLabel 7950 4800 0    60   BiDi ~ 0
 SCL
-Wire Wire Line
-	8550 4050 8250 4050
-Wire Wire Line
-	8250 4050 8250 5100
-Wire Wire Line
-	8250 5100 8950 5100
-Connection ~ 8550 4050
-$Comp
-L GND #PWR4
+$Comp
+L GND #PWR012
 U 1 1 58AEEE1E
-P 2800 1850
-F 0 "#PWR4" H 2800 1600 50  0001 C CNN
-F 1 "GND" H 2800 1700 50  0000 C CNN
-F 2 "" H 2800 1850 50  0000 C CNN
-F 3 "" H 2800 1850 50  0000 C CNN
-	1    2800 1850
-	1    0    0    -1
-$EndComp
-Wire Wire Line
-	2000 1750 2000 2100
-$Comp
-L VCC #PWR1
+P 3500 1900
+F 0 "#PWR012" H 3500 1650 50  0001 C CNN
+F 1 "GND" H 3500 1750 50  0000 C CNN
+F 2 "" H 3500 1900 50  0000 C CNN
+F 3 "" H 3500 1900 50  0000 C CNN
+	1    3500 1900
+	1    0    0    -1
+$EndComp
+Wire Wire Line
+	2700 1800 2700 2150
+$Comp
+L VCC #PWR013
 U 1 1 58AEEFF6
-P 2400 2000
-F 0 "#PWR1" H 2400 1850 50  0001 C CNN
-F 1 "VCC" H 2400 2150 50  0000 C CNN
-F 2 "" H 2400 2000 50  0000 C CNN
-F 3 "" H 2400 2000 50  0000 C CNN
-	1    2400 2000
-	1    0    0    -1
-$EndComp
-Text Label 1200 1450 2    60   ~ 0
+P 3100 2050
+F 0 "#PWR013" H 3100 1900 50  0001 C CNN
+F 1 "VCC" H 3100 2200 50  0000 C CNN
+F 2 "" H 3100 2050 50  0000 C CNN
+F 3 "" H 3100 2050 50  0000 C CNN
+	1    3100 2050
+	1    0    0    -1
+$EndComp
+Text Label 1900 1500 2    60   ~ 0
 VIN
 Wire Wire Line
-	1200 1450 1600 1450
-Wire Wire Line
-	2400 1450 2800 1450
+	1900 1500 2300 1500
+Wire Wire Line
+	3100 1500 3500 1500
 Wire Wire Line
 	4100 4350 4100 4800
@@
 L MC33269 U1
 U 1 1 58B6409C
-P 2000 1500
-F 0 "U1" H 1800 1700 50  0000 C CNN
-F 1 "MC33269" H 2000 1700 50  0000 L CNN
-F 2 "tapMatrix_Shield:SOT223_318H" H 2000 1600 50  0000 C CIN
-F 3 "" H 2000 1500 50  0000 C CNN
-	1    2000 1500
-	1    0    0    -1
-$EndComp
-Wire Wire Line
-	2000 2100 2400 2100
-Wire Wire Line
-	2400 2100 2400 2000
-Wire Wire Line
-	2800 1450 2800 1850
-Connection ~ 2650 1450
+P 2700 1550
+F 0 "U1" H 2500 1750 50  0000 C CNN
+F 1 "MC33269" H 2700 1750 50  0000 L CNN
+F 2 "tapMatrix_Shield:SOT223_318H" H 2700 1650 50  0000 C CIN
+F 3 "" H 2700 1550 50  0000 C CNN
+	1    2700 1550
+	1    0    0    -1
+$EndComp
+Wire Wire Line
+	2700 2150 3100 2150
+Wire Wire Line
+	3100 2150 3100 2050
+Wire Wire Line
+	3500 1500 3500 1900
+Connection ~ 3350 1500
 Wire Wire Line
 	6550 3700 6300 3700
@@
 F 0 "R6" V 1380 2950 50  0000 C CNN
 F 1 "10K" V 1300 2950 50  0000 C CNN
-F 2 "" V 1230 2950 50  0000 C CNN
+F 2 "" V 1230 2950 50  0001 C CNN
 F 3 "" H 1300 2950 50  0000 C CNN
 	1    1300 2950
@@
 	1300 3100 1300 3350
 Connection ~ 1300 3350
+Wire Wire Line
+	4050 2550 4400 2550
+Connection ~ 4050 2350
+Wire Wire Line
+	8550 3950 8550 4200
+$Comp
+L BARREL_JACK CON2
+U 1 1 58BF5CCB
+P 1050 1000
+F 0 "CON2" H 1050 1250 50  0000 C CNN
+F 1 "BARREL_JACK" H 1050 800 50  0000 C CNN
+F 2 "Connectors:BARREL_JACK" H 1050 1000 50  0001 C CNN
+F 3 "" H 1050 1000 50  0000 C CNN
+	1    1050 1000
+	1    0    0    -1
+$EndComp
+$Comp
+L GND #PWR014
+U 1 1 58BF5E25
+P 1550 1200
+F 0 "#PWR014" H 1550 950 50  0001 C CNN
+F 1 "GND" H 1550 1050 50  0000 C CNN
+F 2 "" H 1550 1200 50  0000 C CNN
+F 3 "" H 1550 1200 50  0000 C CNN
+	1    1550 1200
+	1    0    0    -1
+$EndComp
+Wire Wire Line
+	1350 1100 1550 1100
+Wire Wire Line
+	1550 1100 1550 1200
+Wire Wire Line
+	1350 900  1550 900
+Wire Wire Line
+	1550 900  1550 700
+Text Label 1550 700  2    60   ~ 0
+VIN
+Text Label 9250 1250 2    60   ~ 0
+VIN
 $EndSCHEMATC
